Commit message: Добавлена актуальная модель робота

File: src/armbot_description/urdf/dobot.urdf (robot description, URDF)
Before this commit: robot dobot, 6 links, 5 joints
Links:
- removed link link2
- removed link link3
- removed link link4
- removed link link5
- added link link_1; collision mesh filename=package://armbot_description/meshes/link_1.STL; visual mesh filename=package://armbot_description/meshes/link_1.dae
- added link link_2; collision mesh filename=package://armbot_description/meshes/link_2.STL; visual mesh filename=package://armbot_description/meshes/link_2.dae
- added link link_3; collision mesh filename=package://armbot_description/meshes/link_3.dae; visual mesh filename=package://armbot_description/meshes/link_3.dae
- added link link_4; collision mesh filename=package://armbot_description/meshes/link_4.STL; visual mesh filename=package://armbot_description/meshes/link_4.STL
- added link link_end; collision mesh filename=package://armbot_description/meshes/link_end.STL; visual mesh filename=package://armbot_description/meshes/link_end.STL
- added link link_grip; collision mesh filename=package://armbot_description/meshes/link_grip.STL; visual mesh filename=package://armbot_description/meshes/link_grip.STL
- link base_link: mass 1.0 -> None; geometry collision mesh filename=package://armbot_description/meshes/base_link.STL; visual mesh filename=package://armbot_description/meshes/base_link.STL
Joints:
- removed joint joint12
- removed joint joint23
- removed joint joint34
- removed joint joint45
- added joint joint_1: type revolute, parent base_link, child link_1, origin xyz=0 0 0.024 rpy=0 0 -1.570796325, axis 0 0 1, limit lower=-2.25 upper=2.25 effort=150.0 velocity=3.15
- added joint joint_2: type revolute, parent link_1, child link_2, origin xyz=-0.01175 0 0.114 rpy=1.570796325 0 -1.570796325, axis 0 0 1, limit lower=0 upper=1.570796325 effort=150.0 velocity=3.15
- added joint joint_3: type revolute, parent link_2, child link_3, origin xyz=0.02699 0.13228 -0.01175 rpy=0 3.14159265 0, axis 0 0 1, limit lower=0 upper=1.570796325 effort=150.0 velocity=3.15
- added joint joint_4: type revolute, parent link_3, child link_4, origin xyz=0.07431 -0.12684 0.0 rpy=0 3.14159265 0, axis 0 0 1, limit lower=-3.14159265 upper=3.14159265 effort=150.0 velocity=3.15
- added joint joint_end: type fixed, parent link_4, child link_end, origin xyz=-0.06 0.0 0.0 rpy=1.570796325 0 0, axis 0 0 1, limit lower=-3.14159265 upper=3.14159265 effort=150.0 velocity=3.15
- added joint joint_grip: type revolute, parent link_end, child link_grip, origin xyz=0.0 0.0 0.096 rpy=0 0 0, axis 0 0 1, limit lower=-2.5 upper=2.5 effort=150.0 velocity=3.15

Commit message: Отредактирована модель и скетч.

File: src/armbot_description/urdf/dobot.urdf (robot description, URDF)
Before this commit: robot dobot, 8 links, 7 joints
Joints:
- joint joint_grip: limit lower=-2.5 upper=2.5 effort=150.0 velocity=3.15 -> lower=-1.570796325 upper=1.570796325 effort=150.0 velocity=3.15
