Commit message: Добавлена модель

File: src/armbot_description/urdf/model_default/armbot.gazebo.urdf (robot description, URDF)
Before this commit: robot dobot, 8 links, 7 joints
Links:
- link base_link: geometry collision mesh filename=package://armbot_description/meshes/model_default/base_link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; visual mesh filename=package://armbot_description/meshes/model_default/base_link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
- link link_1: geometry collision mesh filename=package://armbot_description/meshes/model_default/link_1.STL; visual mesh filename=package://armbot_description/meshes/model_default/link_1.dae
- link link_2: geometry collision mesh filename=package://armbot_description/meshes/model_default/link_2.STL; visual mesh filename=package://armbot_description/meshes/model_default/link_2.dae
- link link_3: geometry collision mesh filename=package://armbot_description/meshes/model_default/link_3.dae; visual mesh filename=package://armbot_description/meshes/model_default/link_3.dae
- link link_4: geometry collision mesh filename=package://armbot_description/meshes/model_default/link_4.STL; visual mesh filename=package://armbot_description/meshes/model_default/link_4.STL
- link link_end: geometry collision mesh filename=package://armbot_description/meshes/model_default/link_end.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; visual mesh filename=package://armbot_description/meshes/model_default/link_end.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
- link link_grip: geometry collision mesh filename=package://armbot_description/meshes/model_default/link_grip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; visual mesh filename=package://armbot_description/meshes/model_default/link_grip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

File: src/armbot_description/urdf/model_default/dobot.urdf (robot description, URDF)
Before this commit: robot dobot, 8 links, 7 joints
Links:
- link base_link: geometry collision mesh filename=package://armbot_description/meshes/model_default/base_link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; visual mesh filename=package://armbot_description/meshes/model_default/base_link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
- link link_1: geometry collision mesh filename=package://armbot_description/meshes/model_default/link_1.STL; visual mesh filename=package://armbot_description/meshes/model_default/link_1.dae
- link link_2: geometry collision mesh filename=package://armbot_description/meshes/model_default/link_2.STL; visual mesh filename=package://armbot_description/meshes/model_default/link_2.dae
- link link_3: geometry collision mesh filename=package://armbot_description/meshes/model_default/link_3.dae; visual mesh filename=package://armbot_description/meshes/model_default/link_3.dae
- link link_4: geometry collision mesh filename=package://armbot_description/meshes/model_default/link_4.STL; visual mesh filename=package://armbot_description/meshes/model_default/link_4.STL
- link link_end: geometry collision mesh filename=package://armbot_description/meshes/model_default/link_end.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; visual mesh filename=package://armbot_description/meshes/model_default/link_end.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
- link link_grip: geometry collision mesh filename=package://armbot_description/meshes/model_default/link_grip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; visual mesh filename=package://armbot_description/meshes/model_default/link_grip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
Joints:
- joint joint_4: axis 0 0 1 -> 0 1 0
