Commit message: Обновлена модель

File: src/armbot_description/urdf/model_npoa/armbot.urdf (robot description, URDF)
Before this commit: robot armbot, 8 links, 7 joints
Links:
- removed link link_end
- link base_link: mass None -> 0.271570047216607
- link link_1: mass None -> 0.596914732803133
- link link_2: mass None -> 0.100204717897998
- link link_3: mass None -> 0.0817197840637802
- link link_4: mass None -> 0.0816655051489231
- link link_grip: mass None -> 0.14549649198173
Joints:
- removed joint joint_end
- joint joint_1: axis 0 1 0 -> 0 0 1; limit lower=-2.25 upper=2.25 effort=150.0 velocity=3.15 -> lower=-2.25 upper=2.25 effort=150 velocity=3.15; origin xyz=0 0 0.003 rpy=-1.5708 0 0.014721 -> xyz=0.003 0 0.0155 rpy=0 0 0.0047017
- joint joint_2: limit lower=0 upper=1.570796325 effort=150.0 velocity=3.15 -> lower=0 upper=1.5708 effort=150 velocity=3.15; origin xyz=0 -0.086784 0 rpy=-3.1416 0 0.44762 -> xyz=-0.0027435 0.0155 0.095011 rpy=1.5708 -1.5708 0
- joint joint_3: limit lower=0 upper=1.570796325 effort=150.0 velocity=3.15 -> lower=0 upper=1.5708 effort=150 velocity=3.15; origin xyz=-0.14546 0.11597 -6.7308E-05 rpy=0 0 -1.7541 -> xyz=0.13752 -0.011528 0.0061346 rpy=3.1416 0 -2.8478
- joint joint_4: limit lower=-3.14159265 upper=3.14159265 effort=150.0 velocity=3.15 -> lower=-3.14159265 upper=3.14159265 effort=150 velocity=3.15; origin xyz=0.165 0 0 rpy=0 0 0 -> xyz=0.15964 -0.010744 -0.017433 rpy=0 0 -2.825
- joint joint_grip: axis 0 1 0 -> 0 0 1; limit lower=-1.570796325 upper=1.570796325 effort=150.0 velocity=3.15 -> lower=-1.570796325 upper=1.570796325 effort=150 velocity=3.15; origin xyz=0.035 -0.034 -0.0055 rpy=0 1.6 1.55 -> xyz=0.0060861 0.052412 0.0075 rpy=1.5708 0 1.548; parent link_end -> link_4

Commit message: Обновлена модель

File: src/armbot_description/urdf/model_npoa/armbot.urdf (robot description, URDF)
Before this commit: robot armbot, 7 links, 6 joints
Links:
- added link link_end, mass 0.0720522181905562; collision mesh filename=package://armbot_description/meshes/model_npoa/link_end.STL; visual mesh filename=package://armbot_description/meshes/model_npoa/link_end.STL
- link link_1: mass 0.596914732803133 -> 0.579092466366984
- link link_2: mass 0.100204717897998 -> 0.100204717943486
- link link_3: mass 0.0817197840637802 -> 0.0817197581918697
- link link_4: mass 0.0816655051489231 -> 0.0208066724716135
- link link_grip: mass 0.14549649198173 -> 0.142220620437737
Joints:
- added joint joint_end: type fixed, parent link_4, child link_end, origin xyz=0.21371 0.14219 0.0075 rpy=-3.1416 0 1.7749, axis 0 0 0
- joint joint_1: axis 0 0 1 -> 0 0 -1; origin xyz=0.003 0 0.0155 rpy=0 0 0.0047017 -> xyz=0.003 0 0.0155 rpy=-3.1416 0 -3.1269
- joint joint_2: limit lower=0 upper=1.5708 effort=150 velocity=3.15 -> lower=-1.5708 upper=0 effort=150 velocity=3.15; origin xyz=-0.0027435 0.0155 0.095011 rpy=1.5708 -1.5708 0 -> xyz=0.0027435 0.0155 -0.09502 rpy=1.5708 1.5708 0
- joint joint_3: axis 0 0 1 -> 0.0026029 -0.0096749 0.99995; limit lower=0 upper=1.5708 effort=150 velocity=3.15 -> lower=-1.5708 upper=0 effort=150 velocity=3.15; origin xyz=0.13752 -0.011528 0.0061346 rpy=3.1416 0 -2.8478 -> xyz=0.13709 -0.015779 0.0061346 rpy=3.1416 0 -2.8788
- joint joint_4: origin xyz=0.15964 -0.010744 -0.017433 rpy=0 0 -2.825 -> xyz=0.15162 -0.051106 -0.017433 rpy=0 0 -3.0829
- joint joint_grip: axis 0 0 1 -> 0 0 -1; origin xyz=0.0060861 0.052412 0.0075 rpy=1.5708 0 1.548 -> xyz=-0.043378 -0.23321 0 rpy=1.5708 0 0; parent link_4 -> link_end

Commit message: Доработана модель. Сформирована конфигурация

File: src/armbot_description/urdf/model_npoa/armbot.urdf (robot description, URDF)
Before this commit: robot armbot, 8 links, 7 joints
Links:
- link link_grip: geometry collision cylinder length=0.10 radius=0.0025; visual cylinder length=0.10 radius=0.0025
Joints:
- joint joint_end: origin xyz=0.21371 0.14219 0.0075 rpy=-3.1416 0 1.7749 -> xyz=0 0 0 rpy=-3.1416 0 1.7749
- joint joint_grip: origin xyz=-0.043378 -0.23321 0 rpy=1.5708 0 0 -> xyz=0.0525 -0.083 -0.0075 rpy=1.5708 0 0
