Commit message: Добавлена модель робота. Исправлена проблема с загрузкой конфигов.

File: src/armbot_description/urdf/model_best/armbot.urdf (robot description, URDF)
Before this commit: robot armbot_description, 6 links, 5 joints
Links:
- added link link_end, mass 0.0563600278018004; collision mesh filename=package://armbot_description/meshes/model_best/link_end.STL; visual mesh filename=package://armbot_description/meshes/model_best/link_end.STL
- added link link_grip, mass 0.0557728067893349; collision cylinder length=0.10 radius=0.0025; visual cylinder length=0.10 radius=0.0025
- link base_link: mass 0.637079960483491 -> 0.539924220844728
- link link_1: mass 3.72114813626533 -> 3.66151948541535
- link link_2: mass 0.339889695657714 -> 0.270091528613745
- link link_3: mass 0.145541850057218 -> 0.138752300390972
- link link_4: mass 0.115776682365261 -> 0.0428002294983427
Joints:
- added joint joint_end: type fixed, parent link_4, child link_end, origin xyz=0 0 0 rpy=0 0 0, axis 0 0 0
- added joint joint_grip: type revolute, parent link_end, child link_grip, origin xyz=0.037918 -0.021328 -0.0715 rpy=3.1416 0 0, axis 0 0 1, limit lower=-1.570796325 upper=1.570796325 effort=150 velocity=3.15
- joint joint_1: axis 0 1 0 -> 0 0 1; origin xyz=0.036 0 0.023 rpy=1.5708 0 1.5708 -> xyz=0 0 0.023 rpy=0 0 0
- joint joint_2: axis 0 0 -1 -> 0 0 1; limit lower=0 upper=1.5708 effort=150 velocity=3.15 -> lower=0 upper=1.570796325 effort=150 velocity=3.15; origin xyz=0.02 0.126 -0.036 rpy=-1.5708 0.060386 -1.5708 -> xyz=0 0.017 0.126 rpy=-1.5708 0 0
- joint joint_3: axis 0 0 -1 -> 0 0 1; limit lower=0 upper=1.570796325 effort=150 velocity=3.15 -> lower=-1.570796325 upper=0 effort=150 velocity=3.15; origin xyz=-0.135 0 0.012 rpy=0 0 1.9075 -> xyz=0.024396 -0.13278 0.011298 rpy=0 0 -1.5026
- joint joint_4: axis 0 0 1 -> 0 1 0; origin xyz=-0.1225 -0.10506 -0.049 rpy=0 0 -0.39709 -> xyz=-0.15035 0.054723 -0.0068996 rpy=1.5708 0 1.5026
