Commit message: Обновление моделей и конфигураций.

File: src/armbot_description/urdf/model_best/armbot.gazebo.urdf (robot description, URDF)
Before this commit: robot armbot, 8 links, 7 joints
Links:
- link link_end: mass 0.0563600278018004 -> 0.0563600278018003
- link link_grip: mass 0.0557728067893349 -> 0.0557728067893351
Joints:
- joint joint_1: axis 0 0 1 -> 0 0 -1
- joint joint_2: limit lower=0 upper=1.570796325 effort=150 velocity=3.15 -> lower=-1.5708 upper=0 effort=150 velocity=3.15; origin xyz=0 0.017 0.126 rpy=-1.5708 0 0 -> xyz=0 0.017 0.126 rpy=1.5708 -1.5708 0
- joint joint_3: limit lower=-1.570796325 upper=0 effort=150 velocity=3.15 -> lower=-1.5708 upper=0 effort=150 velocity=3.15; origin xyz=0.024396 -0.13278 0.011298 rpy=0 0 -1.5026 -> xyz=0.13278 -0.024396 -0.011298 rpy=3.1416 0 -2.8607
- joint joint_4: axis 0 1 0 -> 0 0 1; origin xyz=-0.15035 0.054723 -0.0068996 rpy=1.5708 0 1.5026 -> xyz=0.16 0 -0.0068996 rpy=-3.1416 0 -1.2899
- joint joint_grip: axis 0 0 1 -> 0 0 -1; origin xyz=0.037918 -0.021328 -0.0715 rpy=3.1416 0 3.1416 -> xyz=0.038079 -0.0716 0.021516 rpy=1.5708 0 0

File: src/armbot_description/urdf/model_best/armbot.urdf (robot description, URDF)
Before this commit: robot armbot, 8 links, 7 joints
Links:
- link link_end: mass 0.0563600278018004 -> 0.0563600278018003
- link link_grip: mass 0.0557728067893349 -> 0.0557728067893351
Joints:
- joint joint_1: axis 0 0 1 -> 0 0 -1
- joint joint_2: limit lower=0 upper=1.570796325 effort=150 velocity=3.15 -> lower=-1.5708 upper=0 effort=150 velocity=3.15; origin xyz=0 0.017 0.126 rpy=-1.5708 0 0 -> xyz=0 0.017 0.126 rpy=1.5708 -1.5708 0
- joint joint_3: limit lower=-1.570796325 upper=0 effort=150 velocity=3.15 -> lower=-1.5708 upper=0 effort=150 velocity=3.15; origin xyz=0.024396 -0.13278 0.011298 rpy=0 0 -1.5026 -> xyz=0.13278 -0.024396 -0.011298 rpy=3.1416 0 -2.8607
- joint joint_4: axis 0 1 0 -> 0 0 1; origin xyz=-0.15035 0.054723 -0.0068996 rpy=1.5708 0 1.5026 -> xyz=0.16 0 -0.0068996 rpy=-3.1416 0 -1.2899
- joint joint_grip: axis 0 0 1 -> 0 0 -1; origin xyz=0.037918 -0.021328 -0.0715 rpy=3.1416 0 0 -> xyz=0.038079 -0.0716 0.021516 rpy=1.5708 0 0

File: src/armbot_description/urdf/model_npoa/armbot.gazebo.urdf (robot description, URDF)
Before this commit: robot armbot, 8 links, 7 joints
Links:
- link link_2: mass 0.100204717943486 -> 0.100204717943485
- link link_3: mass 0.0817197581918697 -> 0.0817197581918649
- link link_grip: geometry collision cylinder length=0.10 radius=0.0025; visual cylinder length=0.10 radius=0.0025
Joints:
- joint joint_1: origin xyz=0.003 0 0.0155 rpy=-3.1416 0 -3.1269 -> xyz=0.003 0 0.0155 rpy=0 0 0
- joint joint_2: axis 0 0 1 -> 0 0.010019 0.99995; origin xyz=0.0027435 0.0155 -0.09502 rpy=1.5708 1.5708 0 -> xyz=0.0026508 0.015956 0.09502 rpy=1.5708 -1.5708 0
- joint joint_4: axis 0 0 1 -> 0 0 -1; origin xyz=0.15162 -0.051106 -0.017433 rpy=0 0 -3.0829 -> xyz=0.15162 -0.051106 -0.017433 rpy=3.1416 0 -1.0232
- joint joint_end: origin xyz=0 0 0 rpy=-3.1416 0 1.7749 -> xyz=0 0 0 rpy=0 0 0
- joint joint_grip: origin xyz=0.0525 -0.0378 -0.0075 rpy=1.5708 0 0 -> xyz=0.0715 -0.064 -0.0075 rpy=1.5708 0 0.27

File: src/armbot_description/urdf/model_npoa/armbot.urdf (robot description, URDF)
Before this commit: robot armbot, 8 links, 7 joints
Links:
- link link_2: mass 0.100204717943486 -> 0.100204717943485
- link link_3: mass 0.0817197581918697 -> 0.0817197581918649
Joints:
- joint joint_1: origin xyz=0.003 0 0.0155 rpy=-3.1416 0 -3.1269 -> xyz=0.003 0 0.0155 rpy=0 0 0
- joint joint_2: axis 0 0 1 -> 0 0.010019 0.99995; origin xyz=0.0027435 0.0155 -0.09502 rpy=1.5708 1.5708 0 -> xyz=0.0026508 0.015956 0.09502 rpy=1.5708 -1.5708 0
- joint joint_4: axis 0 0 1 -> 0 0 -1; origin xyz=0.15162 -0.051106 -0.017433 rpy=0 0 -3.0829 -> xyz=0.15162 -0.051106 -0.017433 rpy=3.1416 0 -1.0232
- joint joint_end: origin xyz=0 0 0 rpy=-3.1416 0 1.7749 -> xyz=0 0 0 rpy=0 0 0
- joint joint_grip: origin xyz=0.0525 -0.083 -0.0075 rpy=1.5708 0 0 -> xyz=0.0715 -0.064 -0.0075 rpy=1.5708 0 0.27

Commit message: Добавлена камера (но пока не работает)

File: src/armbot_description/urdf/model_best/armbot.gazebo.urdf (robot description, URDF)
Before this commit: robot armbot, 8 links, 7 joints
Links:
- added link camera; visual box size=.05 .05 .05
Joints:
- added joint camera_joint: type fixed, parent base_link, child camera, origin xyz=0.3 0 0 rpy=0 0 0

Commit message: Доработка робота для Gazebo

File: src/armbot_description/urdf/model_best/armbot.gazebo.urdf (robot description, URDF)
Before this commit: robot armbot, 9 links, 8 joints
Links:
- link camera: geometry visual box size=.01 .01 .01
Joints:
- joint camera_joint: origin xyz=0.3 0 0 rpy=0 0 0 -> xyz=0.06 -0.0212 0.0205 rpy=0 0 0; parent base_link -> link_end

Commit message: Конфиги для симулятора

File: src/armbot_description/urdf/model_best/armbot.gazebo.urdf (robot description, URDF)
Before this commit: robot armbot, 9 links, 8 joints
Links:
- removed link link_grip
Joints:
- removed joint joint_grip

Commit message: Добавлены контроллеры для запуска в Gazebo

File: src/armbot_description/urdf/model_best/armbot.gazebo.urdf (robot description, URDF)
Before this commit: robot armbot, 8 links, 7 joints
Links:
- added link link_grip, mass 0.0557728067893351; collision cylinder length=0.10 radius=0.0025; visual cylinder length=0.10 radius=0.0025
Joints:
- added joint joint_grip: type revolute, parent link_end, child link_grip, origin xyz=0.038079 -0.0716 0.021516 rpy=1.5708 0 0, axis 0 0 -1, limit lower=-1.570796325 upper=1.570796325 effort=150 velocity=3.15

Commit message: Движение робота в Gazebo

File: src/armbot_description/urdf/model_best/armbot.gazebo.urdf (robot description, URDF)
Before this commit: robot armbot, 9 links, 8 joints
Links:
- link link_2: mass 0.270091528613745 -> 1.2
- link link_4: mass 0.0428002294983427 -> 0.08
- link link_end: mass 0.0563600278018003 -> 0.040
- link link_grip: mass 0.0557728067893351 -> 0.01

Commit message: Корректировка параметров для стабилизации работы.

File: src/armbot_description/urdf/model_best/armbot.gazebo.urdf (robot description, URDF)
Before this commit: robot armbot, 9 links, 8 joints
Links:
- link link_grip: geometry collision cylinder length=0.07 radius=0.0025; visual cylinder length=0.07 radius=0.0025
Joints:
- joint joint_grip: origin xyz=0.038079 -0.0716 0.021516 rpy=1.5708 0 0 -> xyz=0.038079 -0.057 0.021516 rpy=1.5708 0 0

File: src/armbot_description/urdf/model_best/armbot.urdf (robot description, URDF)
Before this commit: robot armbot, 8 links, 7 joints
Links:
- link link_grip: geometry collision cylinder length=0.07 radius=0.0025; visual cylinder length=0.07 radius=0.0025
Joints:
- joint joint_grip: origin xyz=0.038079 -0.0716 0.021516 rpy=1.5708 0 0 -> xyz=0.038079 -0.057 0.021516 rpy=1.5708 0 0

Commit message: Доработка для Gazebo. Вернула стол

File: src/armbot_description/urdf/model_best/armbot.gazebo.urdf (robot description, URDF)
Before this commit: robot armbot, 9 links, 8 joints
Links:
- link link_2: mass 1.2 -> 0.270091528613745
- link link_4: mass 0.08 -> 0.0428002294983427
- link link_end: mass 0.040 -> 0.0563600278018004
- link link_grip: geometry collision cylinder length=0.05 radius=0.0025; visual cylinder length=0.05 radius=0.0025
Joints:
- joint joint_grip: origin xyz=0.038079 -0.057 0.021516 rpy=1.5708 0 0 -> xyz=0.038079 -0.037 0.021516 rpy=1.5708 0 0

Commit message: Добавлена вторая камера на рабочий орган.

File: src/armbot_description/urdf/model_best/armbot.gazebo.urdf (robot description, URDF)
Before this commit: robot armbot, 10 links, 9 joints
Links:
- removed link camera
- added link camera_left; visual box size=.01 .01 .01
- added link camera_right; visual box size=.01 .01 .01
Joints:
- removed joint camera_joint
- added joint camera_left_joint: type fixed, parent link_end, child camera_left, origin xyz=0.06 -0.0212 0.027 rpy=0 0 0
- added joint camera_right_joint: type fixed, parent link_end, child camera_right, origin xyz=0.06 -0.0212 0.016 rpy=0 0 0

Commit message: Добавлена камера глубины.

File: src/armbot_description/urdf/model_best/armbot.gazebo.urdf (robot description, URDF)
Before this commit: robot armbot, 11 links, 10 joints
Joints:
- joint camera_left_joint: origin xyz=0.06 -0.0212 0.027 rpy=0 0 0 -> xyz=0.06 -0.0212 0.016 rpy=0 0 0
- joint camera_right_joint: origin xyz=0.06 -0.0212 0.016 rpy=0 0 0 -> xyz=0.06 -0.0212 0.027 rpy=0 0 0
