Commit message: Добавление клавиатуры

File: src/keyboard_description/urdf/keyboard.xacro (robot description, xacro)
@@ -4,6 +4,12 @@
     <inertial>
         <origin xyz="0.539039 0 0" rpy="1.5708 3.14 1.5708" />
-        <mass value="0.0557728067893351" />
-        <inertia ixx="3.92728176216146E-06" ixy="-2.61102891000333E-12" ixz="3.15138580124161E-07" iyy="5.88583553323269E-06" iyz="9.57169867073918E-11" izz="3.24790074280288E-06" />
+        <mass value="0.56" />
+        <inertia
+          ixx="0.00000024458"
+          ixy="0.00000000002"
+          ixz="0.00000000225"
+          iyy="0.00000221535"
+          iyz="0.00000000113"
+          izz="0.00000196415" />
     </inertial>
     <visual>

Commit message: Добавлена клавиатура для Gazebo.

File: src/keyboard_description/urdf/keyboard.xacro (robot description, xacro)
@@ -1,31 +1,50 @@
-<?xml version="1.0" encoding="utf-8" ?>
-<robot name="keyboard" xmlns:xacro="http://www.ros.org/wiki/xacro">
-  <link name='base'>
+<?xml version="1.0" encoding="utf-8"?>
+<!-- This URDF was automatically created by SolidWorks to URDF Exporter! Originally created by Stephen Brawner (brawner@gmail.com)
+     Commit Version: 1.6.0-4-g7f85cfe  Build Version: 1.6.7995.38578
+     For more information, please see http://wiki.ros.org/sw_urdf_exporter -->
+<robot
+  name="keyboard">
+  <link
+    name="base">
     <inertial>
-        <origin xyz="0.539039 0 0" rpy="1.5708 3.14 1.5708" />
-        <mass value="0.56" />
-        <inertia
-          ixx="0.00000024458"
-          ixy="0.00000000002"
-          ixz="0.00000000225"
-          iyy="0.00000221535"
-          iyz="0.00000000113"
-          izz="0.00000196415" />
+      <origin
+        xyz="0.20298913431108743 0.004842857231127 -0.00965568277916037"
+        rpy="0 0 -1.570796325" />
+      <mass
+        value="0.600478305590293" />
+      <inertia
+        ixx="0.000998570477714973"
+        ixy="-6.45011254701907E-06"
+        ixz="2.21581605764142E-05"
+        iyy="0.00680233708746064"
+        iyz="-2.33214552616074E-05"
+        izz="0.00581941436503155" />
     </inertial>
     <visual>
-      <origin xyz="0.539039 0 0" rpy="1.5708 3.14 1.5708"/>
+      <origin
+        xyz="0.2 0 0"
+        rpy="0 0 -1.570796325" />
       <geometry>
-          <mesh filename="package://keyboard_description/meshes/keyboard.stl" />
+        <mesh
+          filename="package://keyboard_description/meshes/keyboard_gazebo.STL" />
       </geometry>
+      <material
+        name="">
+        <color
+          rgba="0.752941176470588 0.752941176470588 0.752941176470588 1" />
+      </material>
     </visual>
     <collision>
-        <origin xyz="0.539039 0 0" rpy="1.5708 3.14 1.5708" />
-        <geometry>
-            <mesh filename="package://keyboard_description/meshes/keyboard.stl" />
-        </geometry>
+      <origin
+        xyz="0.2 0 0"
+        rpy="0 0 -1.570796325" />
+      <geometry>
+        <mesh
+          filename="package://keyboard_description/meshes/keyboard_gazebo.STL" />
+      </geometry>
     </collision>
   </link>
   <gazebo reference="base">
-      <material>Gazebo/DarkGrey</material>
+      <material>Gazebo/BlackTransparent</material>
   </gazebo>
 </robot>
