Commit message: Gazebo. Доработана сцена симуляции

File: src/armbot_camera/urdf/camera.xacro (robot description, xacro)
@@ -3,5 +3,5 @@
   <xacro:property name="M_PI" value="3.1415926535897931" />
   <static>true</static>
-  <origin xyz="0 0 1.0" rpy=" 0 1.57079633 0"/>
+  <origin xyz="0 0 2.0" rpy=" 0 1.57079633 0"/>
   <xacro:include filename="$(find armbot_camera)/urdf/camera.gazebo" />
   <xacro:include filename="$(find armbot_description)/urdf/materials/materials.xacro" />

Commit message: Реализовано слежение за рабочим органом

File: src/armbot_camera/urdf/camera.xacro (robot description, xacro)
@@ -3,5 +3,5 @@
   <xacro:property name="M_PI" value="3.1415926535897931" />
   <static>true</static>
-  <origin xyz="0 0 2.0" rpy=" 0 1.57079633 0"/>
+  <origin xyz="0 0 1.7" rpy=" 0 1.57079633 0"/>
   <xacro:include filename="$(find armbot_camera)/urdf/camera.gazebo" />
   <xacro:include filename="$(find armbot_description)/urdf/materials/materials.xacro" />

Commit message: Расчет joint_1, добавлен маркер для определения положения раб органа, прочие правки

File: src/armbot_camera/urdf/camera.xacro (robot description, xacro)
@@ -3,5 +3,5 @@
   <xacro:property name="M_PI" value="3.1415926535897931" />
   <static>true</static>
-  <origin xyz="0 0 1.7" rpy=" 0 1.57079633 0"/>
+  <origin xyz="0 0 1.75" rpy=" 0 1.57079633 0"/>
   <xacro:include filename="$(find armbot_camera)/urdf/camera.gazebo" />
   <xacro:include filename="$(find armbot_description)/urdf/materials/materials.xacro" />

File: src/armbot_description/urdf/model_best/armbot.gazebo.urdf (robot description, URDF)
Before this commit: robot armbot, 9 links, 8 joints
Links:
- added link link_grip_marker, mass 0.0001; collision cylinder length=0.001 radius=0.007; visual cylinder length=0.001 radius=0.007
Joints:
- added joint joint_grip_marker: type revolute, parent link_end, child link_grip_marker, origin xyz=0.038079 0.011 0.021516 rpy=1.5708 0 0, axis 0 0 -1, limit lower=-1.570796325 upper=1.570796325 effort=150 velocity=3.15

Commit message: Добавлена 3 камера

File: src/armbot_camera/urdf/camera.xacro (robot description, xacro)
@@ -31,16 +31,30 @@
     </visual>
   </link>
-  <link name='camera'>
+  <link name='camera_1'>
     <visual name='camera_visual'>
       <origin xyz="0 0 0" rpy=" 0 0 0"/>
       <geometry>
-        <box size=".05 .05 .05"/>
+        <box size=".015 .015 .015"/>
       </geometry>
       <material name="gray"/>
     </visual>
   </link>
-  <joint type="fixed" name="camera_joint">
+  <joint type="fixed" name="camera_joint_1">
     <origin xyz="0.15 0 0" rpy="0 0 0"/>
-    <child link="camera"/>
+    <child link="camera_1"/>
+    <parent link="base"/>
+  </joint>
+  <link name='camera_2'>
+    <visual name='camera_visual'>
+      <origin xyz="0 0 0" rpy=" 0 0 0"/>
+      <geometry>
+        <box size=".015 .015 .015"/>
+      </geometry>
+      <material name="gray"/>
+    </visual>
+  </link>
+  <joint type="fixed" name="camera_joint_2">
+    <origin xyz="0.15 0.03 0" rpy="0 0 0"/>
+    <child link="camera_2"/>
     <parent link="base"/>
   </joint>
